File: jumbo-s3/jumbo-s3.kicad_pcb (KiCad board)
At the start: 4 copper layers, 38 x 25 mm, 26 parts, among them J1 GPIO, J2 DEBUG, U1 ESP32-S3, U2 APS12808L-3OBM-BA, Y1 40MHz 10ppm

Commit message: Rev 2.1: unify headers
Parts:
- removed J2: DEBUG, Connector_PinHeader_1.27mm:PinHeader_2x08_P1.27mm_Vertical_SMD
- J1: value GPIO -> Conn_02x22_Odd_Even; footprint Connector_PinHeader_1.27mm:PinHeader_2x15_P1.27mm_Vertical_SMD -> Connector_PinHeader_1.27mm:PinHeader_2x22_P1.27mm_Vertical_SMD
- moved J1 4.45 mm to (163.8, 119.5)
- moved C6 0.41 mm to (158.2, 121.4)
Connections:
- J1 pad 14: GND -> +3.3V
- J1 pad 29: GND -> TxD
- J1 pad 30: GND -> RxD
Routing:
- net EN: track 28.1 -> 51.7 mm
- net GPIO41: track 2.21 -> 22.7 mm, vias 1 -> 2
- net GPIO45: track 1.89 -> 21.7 mm, vias 1 -> 2
- net GPIO39: track 4.19 -> 24.0 mm, vias 1 -> 2
- net GPIO42: track 2.93 -> 21.2 mm, vias 1 -> 2
- net GPIO38: track 4.71 -> 22.5 mm, vias 1 -> 2
- net GPIO40: track 4.10 -> 21.4 mm, vias 1 -> 2
- net GPIO46: track 2.40 -> 19.2 mm
- net GPIO0: track 29.4 -> 13.4 mm, vias 3 -> 1
- net RxD: track 5.00 -> 19.4 mm, vias 2 -> 1
- net TxD: track 4.50 -> 15.7 mm
- net +3.3V: track 21.3 -> 25.3 mm
- net GPIO48: track 11.2 -> 13.7 mm
- net GND: track 18.9 -> 17.6 mm, vias 72 -> 118
- net GPIO47: track 15.1 -> 15.7 mm
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