File: jumbo-s3/jumbo-s3.kicad_pcb (KiCad board)
At the start: 4 copper layers, 38 x 25 mm, 25 parts, among them J1 Conn_02x22_Odd_Even, U1 ESP32-S3, U2 APS12808L-3OBM-BA, Y1 40MHz 10ppm

Commit message: Rev 2.1: final fixes
Parts:
- J1: value Conn_02x22_Odd_Even -> GPIO
Routing:
- net EN: track 51.7 -> 50.1 mm
Changed lines of the file:
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@@
       (effects (font (size 1 1) (thickness 0.15)) (justify mirror))
     )
-    (fp_text value "Conn_02x22_Odd_Even" (at 0 -15.03 270) (layer "B.Fab")
+    (fp_text value "GPIO" (at 0 -15.03 270) (layer "B.Fab")
       (effects (font (size 1 1) (thickness 0.15)) (justify mirror))
     )
@@
   (via (at 158.7 119.575) (size 0.45) (drill 0.2) (layers "F.Cu" "B.Cu") (net 5))
   (segment (start 171.6 134.85) (end 172.25 134.2) (width 0.381) (layer "In2.Cu") (net 5))
+  (segment (start 163.21332 121.185) (end 163.22832 121.2) (width 0.13) (layer "In2.Cu") (net 5))
   (segment (start 171.555804 134.85) (end 171.6 134.85) (width 0.381) (layer "In2.Cu") (net 5))
-  (segment (start 171.685 120.55668) (end 171.685 122.66) (width 0.13) (layer "In2.Cu") (net 5))
-  (segment (start 158.7 119.575) (end 159.24 119.035) (width 0.13) (layer "In2.Cu") (net 5))
+  (segment (start 166.88118 121.2) (end 166.89618 121.185) (width 0.13) (layer "In2.Cu") (net 5))
+  (segment (start 169.568249 122.66) (end 171.685 122.66) (width 0.13) (layer "In2.Cu") (net 5))
   (segment (start 167.755804 138.65) (end 171.555804 134.85) (width 0.381) (layer "In2.Cu") (net 5))
+  (segment (start 168.093249 121.185) (end 169.568249 122.66) (width 0.13) (layer "In2.Cu") (net 5))
   (segment (start 172.25 134.2) (end 172.25 128.75) (width 0.381) (layer "In2.Cu") (net 5))
-  (segment (start 168.442035 119.035) (end 169.392035 119.985) (width 0.13) (layer "In2.Cu") (net 5))
   (segment (start 171.685 122.66) (end 172.25 123.225) (width 0.13) (layer "In2.Cu") (net 5))
-  (segment (start 169.392035 119.985) (end 171.11332 119.985) (width 0.13) (layer "In2.Cu") (net 5))
-  (segment (start 171.11332 119.985) (end 171.685 120.55668) (width 0.13) (layer "In2.Cu") (net 5))
+  (segment (start 166.89618 121.185) (end 168.093249 121.185) (width 0.13) (layer "In2.Cu") (net 5))
+  (segment (start 160.325 121.2) (end 162.77168 121.2) (width 0.13) (layer "In2.Cu") (net 5))
+  (segment (start 163.22832 121.2) (end 166.88118 121.2) (width 0.13) (layer "In2.Cu") (net 5))
+  (segment (start 158.7 119.575) (end 160.325 121.2) (width 0.13) (layer "In2.Cu") (net 5))
   (segment (start 172.25 123.225) (end 172.25 128.75) (width 0.13) (layer "In2.Cu") (net 5))
   (segment (start 156.6 138.65) (end 167.755804 138.65) (width 0.381) (layer "In2.Cu") (net 5))
-  (segment (start 159.24 119.035) (end 168.442035 119.035) (width 0.13) (layer "In2.Cu") (net 5))
+  (segment (start 162.78668 121.185) (end 163.21332 121.185) (width 0.13) (layer "In2.Cu") (net 5))
+  (segment (start 162.77168 121.2) (end 162.78668 121.185) (width 0.13) (layer "In2.Cu") (net 5))
   (segment (start 158.085 121.4) (end 158.7 120.785) (width 0.13) (layer "B.Cu") (net 5))
   (segment (start 158.7 120.785) (end 158.7 119.575) (width 0.13) (layer "B.Cu") (net 5))
@@
   (via (at 151.75 118.025) (size 0.45) (drill 0.2) (layers "F.Cu" "B.Cu") (net 56))
   (via (at 162.8855 131.7) (size 0.5) (drill 0.2) (layers "F.Cu" "B.Cu") (net 56))
-  (segment (start 163.113465 132.864039) (end 161.305719 132.864039) (width 0.13) (layer "In2.Cu") (net 56))
+  (segment (start 151.75 123.30832) (end 151.75 118.025) (width 0.13) (layer "In2.Cu") (net 56))
+  (segment (start 163.113465 132.864039) (end 162.089039 132.864039) (width 0.13) (layer "In2.Cu") (net 56))
+  (segment (start 162.929426 131.7) (end 163.4005 132.171074) (width 0.13) (layer "In2.Cu") (net 56))
+  (segment (start 156.88 127.655) (end 156.09668 127.655) (width 0.13) (layer "In2.Cu") (net 56))
+  (segment (start 163.4005 132.577004) (end 163.113465 132.864039) (width 0.13) (layer "In2.Cu") (net 56))
+  (segment (start 156.09668 127.655) (end 151.75 123.30832) (width 0.13) (layer "In2.Cu") (net 56))
+  (segment (start 162.089039 132.864039) (end 156.88 127.655) (width 0.13) (layer "In2.Cu") (net 56))
+  (segment (start 162.8855 131.7) (end 162.929426 131.7) (width 0.13) (layer "In2.Cu") (net 56))
   (segment (start 163.4005 132.171074) (end 163.4005 132.577004) (width 0.13) (layer "In2.Cu") (net 56))
-  (segment (start 162.8855 131.7) (end 162.929426 131.7) (width 0.13) (layer "In2.Cu") (net 56))
-  (segment (start 151.75 123.30832) (end 151.75 118.025) (width 0.13) (layer "In2.Cu") (net 56))
-  (segment (start 162.929426 131.7) (end 163.4005 132.171074) (width 0.13) (layer "In2.Cu") (net 56))
-  (segment (start 163.4005 132.577004) (end 163.113465 132.864039) (width 0.13) (layer "In2.Cu") (net 56))
-  (segment (start 161.305719 132.864039) (end 151.75 123.30832) (width 0.13) (layer "In2.Cu") (net 56))
   (segment (start 164.057167 132.03) (end 164.54 131.547167) (width 0.13) (layer "F.Cu") (net 57))
   (segment (start 164.54 131.547167) (end 164.54 130.9975) (width 0.13) (layer "F.Cu") (net 57))
